File: _saved_Mother Board.sch (KiCad schematic (older format))
At the start: 103 parts, among them J1 Conn_01x04, J2 USB_B_Mini, J3 Conn_02x05_Odd_Even, J4 Conn_01x04, J5 Conn_01x03, J6 Conn_01x03, J7 Conn_01x04, SW1 SW_Push, U1 SC189, U2 TPS2121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

Commit message: worked on layout of power mux, added inverter to enable 3v3 regulator
Parts:
- gave numbers to parts that had none: 1
Connections:
- net +5V: now also U7.5 (VCC)
Changed lines of the file:
@@
 3v3_REG_OUT
 $Comp
-L logic_mdg:SN74LVC1G04DBVR U?
+L logic_mdg:SN74LVC1G04DBVR U7
 U 1 1 5D954C10
 P 8500 9350
-F 0 "U?" H 8500 9775 50  0000 C CNN
+F 0 "U7" H 8500 9775 50  0000 C CNN
 F 1 "SN74LVC1G04DBVR" H 8500 9684 50  0000 C CNN
 F 2 "Package_TO_SOT_SMD:SOT-23-5_HandSoldering" H 8500 9350 50  0001 C CNN
@@
 NoConn ~ 8150 9150
 $Comp
-L power:GND #PWR?
+L power:GND #PWR0191
 U 1 1 5D9826F2
 P 8150 9550
-F 0 "#PWR?" H 8150 9300 50  0001 C CNN
+F 0 "#PWR0191" H 8150 9300 50  0001 C CNN
 F 1 "GND" H 8155 9377 50  0000 C CNN
 F 2 "" H 8150 9550 50  0001 C CNN
@@
 	0    1    1    0
 $EndComp
+$Comp
+L power:+5V #PWR0229
+U 1 1 5D9849F2
+P 8850 9150
+F 0 "#PWR0229" H 8850 9000 50  0001 C CNN
+F 1 "+5V" V 8850 9350 50  0000 C CNN
+F 2 "" H 8850 9150 50  0001 C CNN
+F 3 "" H 8850 9150 50  0001 C CNN
+	1    8850 9150
+	0    1    1    0
+$EndComp
